File: pxie2529_breakout.sch (KiCad schematic (older format))
At the start: 1 part, among them J1 connector-25x4

Commit message: finished routing
Parts:
- added J2, J3: Conn_02x25_Odd_Even, Connector_IDC:IDC-Header_2x25_P2.54mm_Latch12.0mm_Vertical, symbol Connector_Generic:Conn_02x25_Odd_Even
Connections:
- net B0C0+: now also J3.48 (Pin_48)
- net B0C0-: now also J3.47 (Pin_47)
- net B0C1+: now also J3.46 (Pin_46)
- net B0C1-: now also J3.45 (Pin_45)
- net B0C10+: now also J3.34 (Pin_34)
- net B0C10-: now also J3.33 (Pin_33)
- net B0C11+: now also J3.32 (Pin_32)
- net B0C11-: now also J3.31 (Pin_31)
- net B0C12+: now also J2.37 (Pin_37)
- net B0C12-: now also J2.38 (Pin_38)
- net B0C13+: now also J2.35 (Pin_35)
- net B0C13-: now also J2.36 (Pin_36)
- net B0C14+: now also J2.33 (Pin_33)
- net B0C14-: now also J2.34 (Pin_34)
- net B0C15+: now also J2.31 (Pin_31)
- net B0C15-: now also J2.32 (Pin_32)
- net B0C2+: now also J3.44 (Pin_44)
- net B0C2-: now also J3.43 (Pin_43)
- net B0C3+: now also J3.42 (Pin_42)
- net B0C3-: now also J3.41 (Pin_41)
- net B0C4+: now also J2.47 (Pin_47)
- net B0C4-: now also J2.48 (Pin_48)
- net B0C5+: now also J2.45 (Pin_45)
- net B0C5-: now also J2.46 (Pin_46)
- net B0C6+: now also J2.43 (Pin_43)
- net B0C6-: now also J2.44 (Pin_44)
- net B0C7+: now also J2.41 (Pin_41)
- net B0C7-: now also J2.42 (Pin_42)
- net B0C8+: now also J3.38 (Pin_38)
- net B0C8-: now also J3.37 (Pin_37)
- net B0C9+: now also J3.36 (Pin_36)
- net B0C9-: now also J3.35 (Pin_35)
- net B0R0+: now also J3.50 (Pin_50)
- net B0R0-: now also J3.49 (Pin_49)
- net B0R1+: now also J2.49 (Pin_49)
- net B0R1-: now also J2.50 (Pin_50)
- net B0R2+: now also J3.40 (Pin_40)
- net B0R2-: now also J3.39 (Pin_39)
- net B0R3+: now also J2.39 (Pin_39)
- net B0R3-: now also J2.40 (Pin_40)
- net B1C0+: now also J3.28 (Pin_28)
- net B1C0-: now also J3.27 (Pin_27)
- net B1C1+: now also J3.26 (Pin_26)
- net B1C1-: now also J3.25 (Pin_25)
- net B1C10+: now also J3.14 (Pin_14)
- net B1C10-: now also J3.13 (Pin_13)
- net B1C11+: now also J3.12 (Pin_12)
- net B1C11-: now also J3.11 (Pin_11)
- net B1C12+: now also J2.17 (Pin_17)
- net B1C12-: now also J2.18 (Pin_18)
- net B1C13+: now also J2.15 (Pin_15)
- net B1C13-: now also J2.16 (Pin_16)
- net B1C14+: now also J2.13 (Pin_13)
- net B1C14-: now also J2.14 (Pin_14)
- net B1C15+: now also J2.11 (Pin_11)
- net B1C15-: now also J2.12 (Pin_12)
- net B1C2+: now also J3.24 (Pin_24)
- net B1C2-: now also J3.23 (Pin_23)
- net B1C3+: now also J3.22 (Pin_22)
- net B1C3-: now also J3.21 (Pin_21)
- net B1C4+: now also J2.27 (Pin_27)
- net B1C4-: now also J2.28 (Pin_28)
- net B1C5+: now also J2.25 (Pin_25)
- net B1C5-: now also J2.26 (Pin_26)
- net B1C6+: now also J2.23 (Pin_23)
- net B1C6-: now also J2.24 (Pin_24)
- net B1C7+: now also J2.21 (Pin_21)
- net B1C7-: now also J2.22 (Pin_22)
- net B1C8+: now also J3.18 (Pin_18)
- net B1C8-: now also J3.17 (Pin_17)
- net B1C9+: now also J3.16 (Pin_16)
- net B1C9-: now also J3.15 (Pin_15)
- net B1R0+: now also J3.30 (Pin_30)
- net B1R0-: now also J3.29 (Pin_29)
- net B1R1+: now also J2.29 (Pin_29)
- net B1R1-: now also J2.30 (Pin_30)
- net B1R2+: now also J3.20 (Pin_20)
- net B1R2-: now also J3.19 (Pin_19)
- net B1R3+: now also J2.19 (Pin_19)
- net B1R3-: now also J2.20 (Pin_20)
- net GND: now also J2.2 (Pin_2), J3.2 (Pin_2)
- net TRIGIN: now also J2.1 (Pin_1)
- net TRIGOUT: now also J3.1 (Pin_1)
- no-connect marks 16 -> 32
Other:
- moved on the sheet: J1A, J1B, J1C, J1D

Commit message: fixed connector orientation
Connections:
- net B0C0+: now also J3.3 (Pin_3); no longer J3.48 (Pin_48)
- net B0C0-: now also J3.4 (Pin_4); no longer J3.47 (Pin_47)
- net B0C1+: now also J3.5 (Pin_5); no longer J3.46 (Pin_46)
- net B0C1-: now also J3.6 (Pin_6); no longer J3.45 (Pin_45)
- net B0C10+: now also J3.17 (Pin_17); no longer J3.34 (Pin_34)
- net B0C10-: now also J3.18 (Pin_18); no longer J3.33 (Pin_33)
- net B0C11+: now also J3.19 (Pin_19); no longer J3.32 (Pin_32)
- net B0C11-: now also J3.20 (Pin_20); no longer J3.31 (Pin_31)
- net B0C12+: now also J2.14 (Pin_14); no longer J2.37 (Pin_37)
- net B0C12-: now also J2.13 (Pin_13); no longer J2.38 (Pin_38)
- net B0C13+: now also J2.16 (Pin_16); no longer J2.35 (Pin_35)
- net B0C13-: now also J2.15 (Pin_15); no longer J2.36 (Pin_36)
- net B0C14+: now also J2.18 (Pin_18); no longer J2.33 (Pin_33)
- net B0C14-: now also J2.17 (Pin_17); no longer J2.34 (Pin_34)
- net B0C15+: now also J2.20 (Pin_20); no longer J2.31 (Pin_31)
- net B0C15-: now also J2.19 (Pin_19); no longer J2.32 (Pin_32)
- net B0C2+: now also J3.7 (Pin_7); no longer J3.44 (Pin_44)
- net B0C2-: now also J3.8 (Pin_8); no longer J3.43 (Pin_43)
- net B0C3+: now also J3.9 (Pin_9); no longer J3.42 (Pin_42)
- net B0C3-: now also J3.10 (Pin_10); no longer J3.41 (Pin_41)
- net B0C4+: now also J2.4 (Pin_4); no longer J2.47 (Pin_47)
- net B0C4-: now also J2.3 (Pin_3); no longer J2.48 (Pin_48)
- net B0C5+: now also J2.6 (Pin_6); no longer J2.45 (Pin_45)
- net B0C5-: now also J2.5 (Pin_5); no longer J2.46 (Pin_46)
- net B0C6+: now also J2.8 (Pin_8); no longer J2.43 (Pin_43)
- net B0C6-: now also J2.7 (Pin_7); no longer J2.44 (Pin_44)
- net B0C7+: now also J2.10 (Pin_10); no longer J2.41 (Pin_41)
- net B0C7-: now also J2.9 (Pin_9); no longer J2.42 (Pin_42)
- net B0C8+: now also J3.13 (Pin_13); no longer J3.38 (Pin_38)
- net B0C8-: now also J3.14 (Pin_14); no longer J3.37 (Pin_37)
- net B0C9+: now also J3.15 (Pin_15); no longer J3.36 (Pin_36)
- net B0C9-: now also J3.16 (Pin_16); no longer J3.35 (Pin_35)
- net B0R0+: now also J3.1 (Pin_1); no longer J3.50 (Pin_50)
- net B0R0-: now also J3.2 (Pin_2); no longer J3.49 (Pin_49)
- net B0R1+: now also J2.2 (Pin_2); no longer J2.49 (Pin_49)
- net B0R1-: now also J2.1 (Pin_1); no longer J2.50 (Pin_50)
- net B0R2+: now also J3.11 (Pin_11); no longer J3.40 (Pin_40)
- net B0R2-: now also J3.12 (Pin_12); no longer J3.39 (Pin_39)
- net B0R3+: now also J2.12 (Pin_12); no longer J2.39 (Pin_39)
- net B0R3-: now also J2.11 (Pin_11); no longer J2.40 (Pin_40)
- net B1C0+: now also J3.23 (Pin_23); no longer J3.28 (Pin_28)
- net B1C0-: now also J3.24 (Pin_24); no longer J3.27 (Pin_27)
- net B1C1+: now also J3.25 (Pin_25); no longer J3.26 (Pin_26)
- net B1C1-: now also J3.26 (Pin_26); no longer J3.25 (Pin_25)
- net B1C10+: now also J3.37 (Pin_37); no longer J3.14 (Pin_14)
- net B1C10-: now also J3.38 (Pin_38); no longer J3.13 (Pin_13)
- net B1C11+: now also J3.39 (Pin_39); no longer J3.12 (Pin_12)
- net B1C11-: now also J3.40 (Pin_40); no longer J3.11 (Pin_11)
- net B1C12+: now also J2.34 (Pin_34); no longer J2.17 (Pin_17)
- net B1C12-: now also J2.33 (Pin_33); no longer J2.18 (Pin_18)
- net B1C13+: now also J2.36 (Pin_36); no longer J2.15 (Pin_15)
- net B1C13-: now also J2.35 (Pin_35); no longer J2.16 (Pin_16)
- net B1C14+: now also J2.38 (Pin_38); no longer J2.13 (Pin_13)
- net B1C14-: now also J2.37 (Pin_37); no longer J2.14 (Pin_14)
- net B1C15+: now also J2.40 (Pin_40); no longer J2.11 (Pin_11)
- net B1C15-: now also J2.39 (Pin_39); no longer J2.12 (Pin_12)
- net B1C2+: now also J3.27 (Pin_27); no longer J3.24 (Pin_24)
- net B1C2-: now also J3.28 (Pin_28); no longer J3.23 (Pin_23)
- net B1C3+: now also J3.29 (Pin_29); no longer J3.22 (Pin_22)
- net B1C3-: now also J3.30 (Pin_30); no longer J3.21 (Pin_21)
- net B1C4+: now also J2.24 (Pin_24); no longer J2.27 (Pin_27)
- net B1C4-: now also J2.23 (Pin_23); no longer J2.28 (Pin_28)
- net B1C5+: now also J2.26 (Pin_26); no longer J2.25 (Pin_25)
- net B1C5-: now also J2.25 (Pin_25); no longer J2.26 (Pin_26)
- net B1C6+: now also J2.28 (Pin_28); no longer J2.23 (Pin_23)
- net B1C6-: now also J2.27 (Pin_27); no longer J2.24 (Pin_24)
- net B1C7+: now also J2.30 (Pin_30); no longer J2.21 (Pin_21)
- net B1C7-: now also J2.29 (Pin_29); no longer J2.22 (Pin_22)
- net B1C8+: now also J3.33 (Pin_33); no longer J3.18 (Pin_18)
- net B1C8-: now also J3.34 (Pin_34); no longer J3.17 (Pin_17)
- net B1C9+: now also J3.35 (Pin_35); no longer J3.16 (Pin_16)
- net B1C9-: now also J3.36 (Pin_36); no longer J3.15 (Pin_15)
- net B1R0+: now also J3.21 (Pin_21); no longer J3.30 (Pin_30)
- net B1R0-: now also J3.22 (Pin_22); no longer J3.29 (Pin_29)
- net B1R1+: now also J2.22 (Pin_22); no longer J2.29 (Pin_29)
- net B1R1-: now also J2.21 (Pin_21); no longer J2.30 (Pin_30)
- net B1R2+: now also J3.31 (Pin_31); no longer J3.20 (Pin_20)
- net B1R2-: now also J3.32 (Pin_32); no longer J3.19 (Pin_19)
- net B1R3+: now also J2.32 (Pin_32); no longer J2.19 (Pin_19)
- net B1R3-: now also J2.31 (Pin_31); no longer J2.20 (Pin_20)
- net GND: now also J2.49 (Pin_49), J3.49 (Pin_49); no longer J2.2 (Pin_2), J3.2 (Pin_2)
- net TRIGIN: now also J2.50 (Pin_50); no longer J2.1 (Pin_1)
- net TRIGOUT: now also J3.50 (Pin_50); no longer J3.1 (Pin_1)
Changed lines of the file:
@@
 L Connector_Generic:Conn_02x25_Odd_Even J2
 U 1 1 6255532D
-P 3400 6100
-F 0 "J2" H 3450 7517 50  0000 C CNN
-F 1 "Conn_02x25_Odd_Even" H 3450 7426 50  0000 C CNN
-F 2 "Connector_IDC:IDC-Header_2x25_P2.54mm_Latch12.0mm_Vertical" H 3400 6100 50  0001 C CNN
-F 3 "~" H 3400 6100 50  0001 C CNN
-	1    3400 6100
-	1    0    0    -1
+P 3500 6100
+F 0 "J2" H 3550 7517 50  0000 C CNN
+F 1 "Conn_02x25_Odd_Even" H 3550 7426 50  0000 C CNN
+F 2 "Connector_IDC:IDC-Header_2x25_P2.54mm_Latch12.0mm_Vertical" H 3500 6100 50  0001 C CNN
+F 3 "~" H 3500 6100 50  0001 C CNN
+	1    3500 6100
+	-1   0    0    1
 $EndComp
 $Comp
 L Connector_Generic:Conn_02x25_Odd_Even J3
 U 1 1 6255AC37
-P 4950 6100
-F 0 "J3" H 5000 7517 50  0000 C CNN
-F 1 "Conn_02x25_Odd_Even" H 5000 7426 50  0000 C CNN
-F 2 "Connector_IDC:IDC-Header_2x25_P2.54mm_Latch12.0mm_Vertical" H 4950 6100 50  0001 C CNN
-F 3 "~" H 4950 6100 50  0001 C CNN
-	1    4950 6100
-	1    0    0    -1
+P 5050 6100
+F 0 "J3" H 5100 7517 50  0000 C CNN
+F 1 "Conn_02x25_Odd_Even" H 5100 7426 50  0000 C CNN
+F 2 "Connector_IDC:IDC-Header_2x25_P2.54mm_Latch12.0mm_Vertical" H 5050 6100 50  0001 C CNN
+F 3 "~" H 5050 6100 50  0001 C CNN
+	1    5050 6100
+	-1   0    0    1
 $EndComp
 $Comp
